Commit message: Step 5: Gazebo simulation with diff drive plugin - robot initial drive

File: my_robot_description/urdf/my_robot.urdf.xacro (robot description, xacro)
@@ -49,4 +49,5 @@
     <link name="${name}_wheel_link">
       <visual>
+        <origin xyz="0 0 0" rpy="${pi/2} 0 0"/>
         <geometry>
           <cylinder radius="${wheel_radius}" length="${wheel_width}"/>
@@ -57,4 +58,5 @@
       </visual>
       <collision>
+        <origin xyz="0 0 0" rpy="${pi/2} 0 0"/>
         <geometry>
           <cylinder radius="${wheel_radius}" length="${wheel_width}"/>
@@ -64,5 +66,5 @@
         <mass value="0.3"/>
         <inertia ixx="0.001" iyy="0.001" izz="0.001"
-                 ixy="0"     ixz="0"     iyz="0"/>
+                ixy="0"     ixz="0"     iyz="0"/>
       </inertial>
     </link>
@@ -70,7 +72,8 @@
       <parent link="base_link"/>
       <child  link="${name}_wheel_link"/>
-      <origin xyz="0.1 ${y_reflect * wheel_offset_y} 0" rpy="${-pi/2} 0 0"/>
-      <axis xyz="0 0 1"/>
-    </joint>
+      <origin xyz="0.1 ${y_reflect * wheel_offset_y} 0" rpy="0 0 0"/>
+      <axis xyz="0 1 0"/>
+      <limit effort="10" velocity="10"/>
+  </joint>
   </xacro:macro>
   <!-- ─── Instantiate Wheels ─────────────────────────────── -->
@@ -103,3 +106,30 @@
     <origin xyz="0.3 0 ${-wheel_radius/2}" rpy="0 0 0"/>
   </joint>
+<!-- ─── Wheel Friction ─────────────────────────────────── -->
+  <gazebo reference="left_wheel_link">
+    <mu1>1.0</mu1>
+    <mu2>1.0</mu2>
+  </gazebo>
+  <gazebo reference="right_wheel_link">
+    <mu1>1.0</mu1>
+    <mu2>1.0</mu2>
+  </gazebo>
+  <!-- ─── Gazebo Diff Drive Plugin ──────────────────────────
+       Built-in Gazebo plugin — no ros2_control needed.
+       Subscribes to /cmd_vel and publishes /odom directly.
+  ──────────────────────────────────────────────────────────── -->
+  <gazebo>
+    <plugin filename="gz-sim-diff-drive-system"
+            name="gz::sim::systems::DiffDrive">
+      <left_joint>left_wheel_joint</left_joint>
+      <right_joint>right_wheel_joint</right_joint>
+      <wheel_separation>0.35</wheel_separation>
+      <wheel_radius>0.075</wheel_radius>
+      <odom_publish_frequency>50</odom_publish_frequency>
+      <topic>/model/my_robot/cmd_vel</topic>
+      <odom_topic>odom</odom_topic>
+      <frame_id>odom</frame_id>
+      <child_frame_id>base_footprint</child_frame_id>
+    </plugin>
+  </gazebo>
 </robot>

Commit message: Step 6: PID controller C++ node - compiles and publishes correctly

File: my_robot_description/urdf/my_robot.urdf.xacro (robot description, xacro)
@@ -133,3 +133,41 @@
     </plugin>
   </gazebo>
+  <!-- ─── ros2_control Hardware Interface ───────────────────
+       Defines what each joint exposes to ROS2 controllers:
+       - command_interface velocity: we SEND speed to wheels
+       - state_interface velocity:   we READ wheel speed back
+       - state_interface position:   we READ wheel angle back
+  ──────────────────────────────────────────────────────────── -->
+  <ros2_control name="GazeboSystem" type="system">
+    <hardware>
+      <plugin>gz_ros2_control/GazeboSimSystem</plugin>
+    </hardware>
+    <joint name="left_wheel_joint">
+      <command_interface name="velocity">
+        <param name="min">-10</param>
+        <param name="max">10</param>
+      </command_interface>
+      <state_interface name="velocity"/>
+      <state_interface name="position"/>
+    </joint>
+    <joint name="right_wheel_joint">
+      <command_interface name="velocity">
+        <param name="min">-10</param>
+        <param name="max">10</param>
+      </command_interface>
+      <state_interface name="velocity"/>
+      <state_interface name="position"/>
+    </joint>
+  </ros2_control>
+  <!-- ─── gz_ros2_control Plugin ────────────────────────────
+       Loads inside Gazebo and connects ros2_control to
+       Gazebo's physics engine. The parameters file tells it
+       which controllers to make available.
+  ──────────────────────────────────────────────────────────── -->
+  <gazebo>
+    <plugin filename="gz_ros2_control-system"
+            name="gz_ros2_control::GazeboSimROS2ControlPlugin">
+      <parameters>$(find my_robot_description)/config/ros2_control.yaml</parameters>
+    </plugin>
+  </gazebo>
 </robot>

Commit message: Step 6: PID controller implementation
Changes made:
- Added PID controller C++ node (my_robot_controllers)
- Created pid_controller.hpp header with class definition
- Created pid_controller.cpp with full PID implementation
- Updated CMakeLists.txt and package.xml with dependencies
- Updated gazebo.launch.py: headless mode (-s flag), removed spawners
- Updated URDF: single diff drive plugin, removed gz_ros2_control
- Added topic relay and bridge for /model/my_robot/cmd_vel
- PID publishes directly to /model/my_robot/cmd_vel
- Known issue: WSL2 limits message rate to ~1.5Hz (hardware limitation)

File: my_robot_description/urdf/my_robot.urdf.xacro (robot description, xacro)
@@ -133,41 +133,3 @@
     </plugin>
   </gazebo>
-  <!-- ─── ros2_control Hardware Interface ───────────────────
-       Defines what each joint exposes to ROS2 controllers:
-       - command_interface velocity: we SEND speed to wheels
-       - state_interface velocity:   we READ wheel speed back
-       - state_interface position:   we READ wheel angle back
-  ──────────────────────────────────────────────────────────── -->
-  <ros2_control name="GazeboSystem" type="system">
-    <hardware>
-      <plugin>gz_ros2_control/GazeboSimSystem</plugin>
-    </hardware>
-    <joint name="left_wheel_joint">
-      <command_interface name="velocity">
-        <param name="min">-10</param>
-        <param name="max">10</param>
-      </command_interface>
-      <state_interface name="velocity"/>
-      <state_interface name="position"/>
-    </joint>
-    <joint name="right_wheel_joint">
-      <command_interface name="velocity">
-        <param name="min">-10</param>
-        <param name="max">10</param>
-      </command_interface>
-      <state_interface name="velocity"/>
-      <state_interface name="position"/>
-    </joint>
-  </ros2_control>
-  <!-- ─── gz_ros2_control Plugin ────────────────────────────
-       Loads inside Gazebo and connects ros2_control to
-       Gazebo's physics engine. The parameters file tells it
-       which controllers to make available.
-  ──────────────────────────────────────────────────────────── -->
-  <gazebo>
-    <plugin filename="gz_ros2_control-system"
-            name="gz_ros2_control::GazeboSimROS2ControlPlugin">
-      <parameters>$(find my_robot_description)/config/ros2_control.yaml</parameters>
-    </plugin>
-  </gazebo>
 </robot>

Commit message: feat(description): add IMU link and joint to URDF
IMU link parented to chassis_link (physical body) rather than
base_link (abstract frame). Placement at geometric center of
chassis top surface derived from xacro properties:
  xyz = (base_length/2, 0, base_height/2) = (0.2, 0, 0.075)

Using xacro property expressions directly so placement
auto-updates if chassis dimensions change.

Verified via tf2_echo: chassis_link -> imu_link
  Translation: [0.200, 0.000, 0.075]
  Rotation: [0.000, 0.000, 0.000, 1.000] (identity)

Sensor plugin intentionally excluded — kept in next commit
for hardware/sim separation.

File: my_robot_description/urdf/my_robot.urdf.xacro (robot description, xacro)
@@ -115,4 +115,27 @@
     <mu2>1.0</mu2>
   </gazebo>
+  <!-- ─── IMU ──────────────────────────────────────────────── -->
+  <!-- Mounted at geometric center of chassis top surface       -->
+  <!-- xyz = (base_length/2, 0, base_height/2) = (0.2, 0, 0.075) in chassis_link frame -->
+  <link name="imu_link">
+    <visual>
+      <geometry>
+        <box size="0.05 0.05 0.02"/>
+      </geometry>
+      <material name="red">
+        <color rgba="0.8 0.1 0.1 1.0"/>
+      </material>
+    </visual>
+    <inertial>
+      <mass value="0.01"/>
+      <inertia ixx="1e-6" ixy="0" ixz="0"
+               iyy="1e-6" iyz="0" izz="1e-6"/>
+    </inertial>
+  </link>
+  <joint name="imu_joint" type="fixed">
+    <parent link="chassis_link"/>
+    <child  link="imu_link"/>
+    <origin xyz="${base_length/2} 0 ${base_height/2}" rpy="0 0 0"/>
+  </joint>
   <!-- ─── Gazebo Diff Drive Plugin ──────────────────────────
        Built-in Gazebo plugin — no ros2_control needed.
